File: pcb/display-model-b/base/rev-a/base.sch (EAGLE design)
At the start: 37 parts, among them J1 SNG-2MM-HEADER-07-V, Q1 MMBT3904, Q2 MMBT3904, Q3 MMBT3904, Q4 MMBT3904, U1 PCA9634PW, U2 TSL2561FN, X1 CLOCK_LED_SEGMENT, X2 CLOCK_LED_SEGMENT, X3 CLOCK_LED_SEGMENT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

Commit message: Added Model B drawings
Parts:
- removed D5: {ATTR:COLOR}, Optoelectronic:LED-T1
- removed R17: 82, Passive:RES-0603
- R10, R11, R12: value 2.2k -> (none)
- R13: value 3k -> (none)
- R14: value 82 -> (none)
Connections:
- removed net N$20: D5.A, R17.1
- removed net N$21: D5.K, U1.LED3
- net 3.3V: no longer R17.2
Other:
- moved on the sheet: D4, R14
