File: pcb/display-model-b/digit/digit.brd (EAGLE design)
At the start: 26.7 x 40.6 mm, 55 parts, among them J1 SOLDER_JUMPER_3, J2 SOLDER_JUMPER_3, J3 SOLDER_JUMPER_3, Q1 MMBT3904, Q2 MMBT3904, Q3 MMBT3904, Q4 MMBT3904, Q5 MMBT3904, Q6 MMBT3904, Q7 MMBT3904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

Commit message: Added Model B drawings
Parts:
- R17, R18, R19, R20, R21, R22, R23: value (none) -> 3k
Changed lines of the file:
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@@
 <attribute name="NAME" x="13.589" y="3.556" size="0.8128" layer="26" font="vector" ratio="10" rot="MR270"/>
 </element>
-<element name="R17" library="Passive" package="SMD_0603" value="" x="21.59" y="8.255" smashed="yes" rot="MR180">
+<element name="R17" library="Passive" package="SMD_0603" value="3k" x="21.59" y="8.255" smashed="yes" rot="MR180">
 <attribute name="PACKAGE" value="SMT 0603" x="21.59" y="8.255" size="1.27" layer="28" ratio="12" rot="MR180" display="off"/>
 <attribute name="PART" value="" x="21.59" y="8.255" size="1.27" layer="28" ratio="12" rot="MR180" display="off"/>
@@
 <attribute name="NAME" x="19.685" y="8.255" size="0.8128" layer="26" font="vector" ratio="10" rot="MR0"/>
 </element>
-<element name="R18" library="Passive" package="SMD_0603" value="" x="18.415" y="29.21" smashed="yes" rot="MR270">
+<element name="R18" library="Passive" package="SMD_0603" value="3k" x="18.415" y="29.21" smashed="yes" rot="MR270">
 <attribute name="PACKAGE" value="SMT 0603" x="18.415" y="29.21" size="1.27" layer="28" ratio="12" rot="MR270" display="off"/>
 <attribute name="PART" value="" x="18.415" y="29.21" size="1.27" layer="28" ratio="12" rot="MR270" display="off"/>
@@
 <attribute name="NAME" x="17.399" y="31.115" size="0.8128" layer="26" font="vector" ratio="10" rot="MR270"/>
 </element>
-<element name="R19" library="Passive" package="SMD_0603" value="" x="13.335" y="31.75" smashed="yes" rot="MR0">
+<element name="R19" library="Passive" package="SMD_0603" value="3k" x="13.335" y="31.75" smashed="yes" rot="MR0">
 <attribute name="PACKAGE" value="SMT 0603" x="13.335" y="31.75" size="1.27" layer="28" ratio="12" rot="MR0" display="off"/>
 <attribute name="PART" value="" x="13.335" y="31.75" size="1.27" layer="28" ratio="12" rot="MR0" display="off"/>
@@
 <attribute name="NAME" x="15.621" y="32.766" size="0.8128" layer="26" font="vector" ratio="10" rot="MR0"/>
 </element>
-<element name="R20" library="Passive" package="SMD_0603" value="" x="6.35" y="9.525" smashed="yes" rot="MR270">
+<element name="R20" library="Passive" package="SMD_0603" value="3k" x="6.35" y="9.525" smashed="yes" rot="MR270">
 <attribute name="PACKAGE" value="SMT 0603" x="6.35" y="9.525" size="1.27" layer="28" ratio="12" rot="MR270" display="off"/>
 <attribute name="PART" value="" x="6.35" y="9.525" size="1.27" layer="28" ratio="12" rot="MR270" display="off"/>
@@
 <attribute name="NAME" x="6.5024" y="11.3538" size="0.8128" layer="26" font="vector" ratio="10" rot="MR90"/>
 </element>
-<element name="R21" library="Passive" package="SMD_0603" value="" x="5.08" y="13.335" smashed="yes" rot="MR270">
+<element name="R21" library="Passive" package="SMD_0603" value="3k" x="5.08" y="13.335" smashed="yes" rot="MR270">
 <attribute name="PACKAGE" value="SMT 0603" x="5.08" y="13.335" size="1.27" layer="28" ratio="12" rot="MR270" display="off"/>
 <attribute name="PART" value="" x="5.08" y="13.335" size="1.27" layer="28" ratio="12" rot="MR270" display="off"/>
@@
 <attribute name="NAME" x="4.064" y="15.367" size="0.8128" layer="26" font="vector" ratio="10" rot="MR270"/>
 </element>
-<element name="R22" library="Passive" package="SMD_0603" value="" x="3.81" y="26.035" smashed="yes" rot="MR0">
+<element name="R22" library="Passive" package="SMD_0603" value="3k" x="3.81" y="26.035" smashed="yes" rot="MR0">
 <attribute name="PACKAGE" value="SMT 0603" x="3.81" y="26.035" size="1.27" layer="28" ratio="12" rot="MR0" display="off"/>
 <attribute name="PART" value="" x="3.81" y="26.035" size="1.27" layer="28" ratio="12" rot="MR0" display="off"/>
@@
 <attribute name="NAME" x="1.778" y="27.178" size="0.8128" layer="26" font="vector" ratio="10" rot="MR270"/>
 </element>
-<element name="R23" library="Passive" package="SMD_0603" value="" x="3.175" y="19.685" smashed="yes" rot="MR90">
+<element name="R23" library="Passive" package="SMD_0603" value="3k" x="3.175" y="19.685" smashed="yes" rot="MR90">
 <attribute name="PACKAGE" value="SMT 0603" x="3.175" y="19.685" size="1.27" layer="28" ratio="12" rot="MR90" display="off"/>
 <attribute name="PART" value="" x="3.175" y="19.685" size="1.27" layer="28" ratio="12" rot="MR90" display="off"/>
