File: pcb/display-model-b/digit/digit.sch (EAGLE design)
At the start: 51 parts, among them J1 DL-100-HEADER-02-EDGE, J10 SOLDER_JUMPER_3, J11 SOLDER_JUMPER_3, J2 DL-100-HEADER-02-EDGE, Q1 MMBT3904, Q2 MMBT3904, Q3 MMBT3904, Q4 MMBT3904, Q5 MMBT3904, Q6 MMBT3904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

Commit message: Display base pcb (rev C), Touch panel (rev B)
Parts:
- D1, D10, D11, D12, D13, D14, D2, D3, D4, D7, D8, D9: value Red -> Orange; COLOR Red -> Orange; PART_NO APT2012SECK/J3-PRV -> APT2012SECK/J4-PRV
- D5: COLOR Red -> Orange; PART_NO APT2012SECK/J3-PRV -> APT2012SECK/J4-PRV
- D6: value Red -> orange; COLOR Red -> Orange; PART_NO APT2012SECK/J3-PRV -> APT2012SECK/J4-PRV
- R1, R10, R11, R12, R13, R14, R2, R3, R4, R5, R6, R7, R8, R9: value 56 -> 82

Commit message: Changed page format on schematics to US letter (8.5" x 11")
Other:
- moved on the sheet: C1, D1, D10, D11, D12, D13, D14, D2, D3, D4, D5, D6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
