File: pcb/tests/audio/usbspk.brd (EAGLE design)
At the start: 36.8 x 25.4 mm, 34 parts, among them J1 SNG-100-HEADER-04-HDR-V, J2 SNG-100-HEADER-02-FL-V, Q1 12MHz, SW1 B3F-1020, SW2 B3F-1020, SW3 B3F-1020, U4 PCM2704C, U5 TPA2005D1DGN

Commit message: Corrected drawings of touch panel PCB
Parts:
- C13: value 100uF -> 100uF 10v
- C14, C15: value (none) -> 18pF
- C18: value 1uF -> 1uF 10v
- C19: value 22nF -> 0.022 uF
Changed lines of the file:
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@@
 <layer number="19" name="Unrouted" color="6" fill="1" visible="yes" active="yes"/>
 <layer number="20" name="Dimension" color="15" fill="1" visible="yes" active="yes"/>
-<layer number="21" name="tPlace" color="7" fill="1" visible="no" active="yes"/>
-<layer number="22" name="bPlace" color="7" fill="1" visible="no" active="yes"/>
+<layer number="21" name="tPlace" color="7" fill="1" visible="yes" active="yes"/>
+<layer number="22" name="bPlace" color="7" fill="1" visible="yes" active="yes"/>
 <layer number="23" name="tOrigins" color="15" fill="1" visible="yes" active="yes"/>
 <layer number="24" name="bOrigins" color="15" fill="1" visible="yes" active="yes"/>
-<layer number="25" name="tNames" color="7" fill="1" visible="no" active="yes"/>
-<layer number="26" name="bNames" color="7" fill="1" visible="no" active="yes"/>
+<layer number="25" name="tNames" color="7" fill="1" visible="yes" active="yes"/>
+<layer number="26" name="bNames" color="7" fill="1" visible="yes" active="yes"/>
 <layer number="27" name="tValues" color="7" fill="1" visible="no" active="yes"/>
 <layer number="28" name="bValues" color="7" fill="1" visible="no" active="yes"/>
@@
 <layer number="44" name="Drills" color="7" fill="1" visible="no" active="yes"/>
 <layer number="45" name="Holes" color="7" fill="1" visible="yes" active="yes"/>
-<layer number="46" name="Milling" color="3" fill="1" visible="yes" active="yes"/>
+<layer number="46" name="Milling" color="3" fill="1" visible="no" active="yes"/>
 <layer number="47" name="Measures" color="7" fill="1" visible="no" active="yes"/>
 <layer number="48" name="Document" color="7" fill="1" visible="no" active="yes"/>
@@
 <layer number="112" name="tSilk" color="7" fill="1" visible="no" active="yes"/>
 <layer number="116" name="centerDrill" color="7" fill="1" visible="no" active="yes"/>
-<layer number="121" name="_tsilk" color="14" fill="1" visible="yes" active="yes"/>
-<layer number="122" name="_bsilk" color="5" fill="1" visible="yes" active="yes"/>
+<layer number="121" name="_tsilk" color="14" fill="1" visible="no" active="yes"/>
+<layer number="122" name="_bsilk" color="5" fill="1" visible="no" active="yes"/>
 <layer number="123" name="tTestmark" color="7" fill="1" visible="no" active="yes"/>
 <layer number="124" name="bTestmark" color="7" fill="1" visible="no" active="yes"/>
@@
 <attribute name="NAME" x="31.6992" y="22.9616" size="1.016" layer="25" font="vector" ratio="10" rot="R180"/>
 </element>
-<element name="C13" library="Passive" package="CAP_S1210" value="100uF" x="15.875" y="12.7" smashed="yes" rot="R270">
+<element name="C13" library="Passive" package="CAP_S1210" value="100uF 10v" x="15.875" y="12.7" smashed="yes" rot="R270">
 <attribute name="DESCRIPTION" value="{DESCRIPTION} - SMT 1210 - {VALUE}" x="15.875" y="12.7" size="1.27" layer="27" rot="R270" display="off"/>
 <attribute name="NAME" x="15.24" y="10.16" size="1.016" layer="25" font="vector" ratio="10" rot="R270"/>
@@
 <attribute name="NAME" x="30.099" y="9.271" size="1.016" layer="25" font="vector" ratio="10"/>
 <attribute name="VALUE" x="26.543" y="20.955" size="1.27" layer="27" ratio="10" rot="R270"/>
-</element>
-<element name="C14" library="Passive" package="SMD_0603" value="" x="34.29" y="12.065" smashed="yes" rot="R270">
+<attribute name="MFG" value="TXC" x="30.48" y="15.875" size="1.778" layer="27" rot="R270" display="off"/>
+<attribute name="PART_NO" value="9C-12.000MEEJ-T" x="30.48" y="15.875" size="1.778" layer="27" rot="R270" display="off"/>
+</element>
+<element name="C14" library="Passive" package="SMD_0603" value="18pF" x="34.29" y="12.065" smashed="yes" rot="R270">
 <attribute name="PACKAGE" value="SMT 0603" x="34.29" y="12.065" size="1.27" layer="27" rot="R270" display="off"/>
 <attribute name="DESCRIPTION" value="{DESCRIPTION} - SMT 0603 - {value}" x="34.29" y="12.065" size="1.27" layer="27" rot="R270" display="off"/>
@@
 <attribute name="NAME" x="35.306" y="17.272" size="1.016" layer="25" font="vector" ratio="10" rot="R270"/>
 </element>
-<element name="C15" library="Passive" package="SMD_0603" value="" x="34.29" y="19.685" smashed="yes" rot="R90">
+<element name="C15" library="Passive" package="SMD_0603" value="18pF" x="34.29" y="19.685" smashed="yes" rot="R90">
 <attribute name="PACKAGE" value="SMT 0603" x="34.29" y="19.685" size="1.27" layer="27" rot="R90" display="off"/>
 <attribute name="DESCRIPTION" value="{DESCRIPTION} - SMT 0603 - {value}" x="34.29" y="19.685" size="1.27" layer="27" rot="R90" display="off"/>
@@
 <attribute name="NAME" x="12.065" y="19.812" size="1.016" layer="25" font="vector" ratio="10" rot="R90"/>
 </element>
-<element name="C18" library="Passive" package="CAP_S0805" value="1uF" x="12.065" y="10.795" smashed="yes">
+<element name="C18" library="Passive" package="CAP_S0805" value="1uF 10v" x="12.065" y="10.795" smashed="yes">
 <attribute name="DESCRIPTION" value="{DESCRIPTION} - SMT 0805 - {VALUE}" x="12.065" y="10.795" size="1.27" layer="27" display="off"/>
 <attribute name="NAME" x="12.065" y="8.763" size="1.016" layer="25" font="vector" ratio="10"/>
@@
 <attribute name="NAME" x="12.065" y="7.62" size="1.016" layer="25" font="vector" ratio="10"/>
 </element>
-<element name="C19" library="Passive" package="SMD_0603" value="22nF" x="15.875" y="17.145" smashed="yes" rot="R180">
+<element name="C19" library="Passive" package="SMD_0603" value="0.022 uF" x="15.875" y="17.145" smashed="yes" rot="R180">
 <attribute name="PACKAGE" value="SMT 0603" x="15.875" y="17.145" size="1.27" layer="27" rot="R180" display="off"/>
 <attribute name="DESCRIPTION" value="{DESCRIPTION} - SMT 0603 - {value}" x="15.875" y="17.145" size="1.27" layer="27" rot="R180" display="off"/>
