File: pcb/tests/psu/psu_test.brd (EAGLE design)
At the start: 29.2 x 31.8 mm, 27 parts, among them J1 CUI-PJ-013C, J2 SNG-100-HEADER-05-HDR-V, J3 SNG-100-HEADER-04-HDR-V, J4 SNG-100-HEADER-03-HDR-V, U1 ADP2303ARDZ, U2 TPS62086RLT, U3 TS4040D30IDBZ

Commit message: Corrected drawings of touch panel PCB
Parts:
- C1, C2: value 10uF 50V -> 10uF 25V
- C3: value 100nF -> 100nF 25v
- C4: value 10uF 50v -> 10uF 25v
- C5: value 100uF -> 47uF 10v
- C6: value (none) -> 10uF 25v
- C7: value (none) -> 22uF
- C8: value (none) -> 100nF
- D1: value 40V 3A -> 30V 4A
- L2: value (none) -> 4.7uH
- L3: value (none) -> 470nH
- R2: value 53.6K 1% -> 52.3K 1%
- R3: value 10K 1% -> 10.2K 1%
