File: pcb/display-model-b/dots/dots.brd (EAGLE design)
At the start: 6.3 x 6.3 mm, 4 parts

Commit message: Added Model B drawings
Parts:
- R1: value (none) -> 56
Changed lines of the file:
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@@
 <element name="W1" library="Misc" package="WIRE_SMT" value="" x="1.27" y="3.175" rot="MR90"/>
 <element name="W2" library="Misc" package="WIRE_SMT" value="" x="5.08" y="3.175" rot="MR90"/>
-<element name="R1" library="Passive" package="SMD_0603" value="" x="3.175" y="2.54" smashed="yes" rot="MR90">
+<element name="R1" library="Passive" package="SMD_0603" value="56" x="3.175" y="2.54" smashed="yes" rot="MR90">
 <attribute name="PACKAGE" value="SMT 0603" x="3.175" y="2.54" size="1.27" layer="28" rot="MR90" display="off"/>
 <attribute name="PART" value="" x="3.175" y="2.54" size="1.27" layer="28" rot="MR90" display="off"/>

Commit message: Display base pcb (rev C), Touch panel (rev B)
Parts:
- R1: value 56 -> 82
Changed lines of the file:
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@@
 <attribute name="SKU" value="-" x="3.175" y="3.175" size="1.27" layer="27" rot="R270" display="off"/>
 <attribute name="VALUE" value="{ATTR:COLOR}" x="3.175" y="3.175" size="1.27" layer="27" rot="R270" display="off"/>
-<attribute name="COLOR" value="Green" x="3.175" y="3.175" size="1.27" layer="27" rot="R270" display="off"/>
+<attribute name="COLOR" value="Orange" x="3.175" y="3.175" size="1.27" layer="27" rot="R270" display="off"/>
 <attribute name="NAME" x="1.0922" y="4.3434" size="0.8128" layer="25" font="vector" ratio="10"/>
+<attribute name="PART_NO" value="APT2012SECK/J4-PRV" x="3.175" y="3.175" size="1.778" layer="27" rot="R270" display="off"/>
 </element>
 <element name="W1" library="Misc" package="WIRE_SMT" value="" x="1.27" y="3.175" rot="MR90">
@@
 <attribute name="BOM" value="FALSE" x="5.08" y="3.175" size="1.778" layer="28" rot="MR90" display="off"/>
 </element>
-<element name="R1" library="Passive" package="SMD_0603" value="56" x="3.175" y="2.54" smashed="yes" rot="MR90">
+<element name="R1" library="Passive" package="SMD_0603" value="82" x="3.175" y="2.54" smashed="yes" rot="MR90">
 <attribute name="PACKAGE" value="SMT 0603" x="3.175" y="2.54" size="1.27" layer="28" rot="MR90" display="off"/>
 <attribute name="PART" value="" x="3.175" y="2.54" size="1.27" layer="28" rot="MR90" display="off"/>
