File: pcb/display-model-a/display.brd (EAGLE design)
At the start: 121.9 x 17.8 mm, 64 parts, among them J1 SNG-2MM-HEADER-07-V, Q1 ALS-PT19, U1 PIC16F1826-I/SS, U2 74HC4017D, U3 74HC4017D, U4 74HC4017D, U5 74LVC1G08DCKR, U6 74LVC1G08DCKR

Commit message: Changed page format on schematics to US letter (8.5" x 11")
Connections:
- net N$53 renamed COL1
- net N$70 renamed COL2
- net N$71 renamed COL3
- net N$72 renamed COL4
- net N$73 renamed COL5
- net N$74 renamed COL6
- net N$75 renamed COL7
- net N$76 renamed COL8
- net N$77 renamed COL9
- net N$78 renamed COL10
- net N$79 renamed COL12
- net N$80 renamed COL11
- net N$81 renamed COL13
- net N$82 renamed COL14
- net N$83 renamed COL15
- net N$84 renamed COL16
- net N$85 renamed COL17
- net N$86 renamed COL18
- net N$87 renamed COL19
- net N$88 renamed COL20
- net N$89 renamed COL21
- net N$90 renamed COL22
- net N$91 renamed COL23
- net N$92 renamed COL24
Changed lines of the file:
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@@
 <layer number="44" name="Drills" color="7" fill="1" visible="no" active="yes"/>
 <layer number="45" name="Holes" color="7" fill="1" visible="yes" active="yes"/>
-<layer number="46" name="Milling" color="3" fill="1" visible="yes" active="yes"/>
+<layer number="46" name="Milling" color="3" fill="1" visible="no" active="yes"/>
 <layer number="47" name="Measures" color="7" fill="1" visible="no" active="yes"/>
 <layer number="48" name="Document" color="7" fill="1" visible="no" active="yes"/>
@@
 <wire x1="86.36" y1="3.81" x2="84.67" y2="3.81" width="0.254" layer="16"/>
 </signal>
-<signal name="N$53">
+<signal name="COL1">
 <contactref element="R10" pad="1"/>
 <contactref element="U4" pad="2"/>
@@
 <wire x1="10.795" y1="8.675" x2="10.795" y2="7.62" width="0.254" layer="16"/>
 </signal>
-<signal name="N$70">
+<signal name="COL2">
 <contactref element="U4" pad="4"/>
 <contactref element="R11" pad="1"/>
@@
 <wire x1="10.16" y1="8.89" x2="5.295" y2="8.89" width="0.254" layer="1"/>
 </signal>
-<signal name="N$71">
+<signal name="COL3">
 <contactref element="R12" pad="1"/>
 <contactref element="U4" pad="7"/>
@@
 <wire x1="18.835" y1="8.675" x2="19.05" y2="8.89" width="0.254" layer="16"/>
 </signal>
-<signal name="N$72">
+<signal name="COL4">
 <contactref element="U4" pad="10"/>
 <contactref element="R13" pad="1"/>
 <wire x1="18.288" y1="8.89" x2="15.455" y2="8.89" width="0.254" layer="1"/>
 </signal>
-<signal name="N$73">
+<signal name="COL5">
 <contactref element="R14" pad="1"/>
 <contactref element="U4" pad="1"/>
@@
 <wire x1="26.67" y1="2.54" x2="26.67" y2="5.5" width="0.254" layer="16"/>
 </signal>
-<signal name="N$74">
+<signal name="COL6">
 <contactref element="U4" pad="5"/>
 <contactref element="R15" pad="1"/>
@@
 <wire x1="22.01" y1="8.675" x2="20.955" y2="7.62" width="0.254" layer="16"/>
 </signal>
-<signal name="N$75">
+<signal name="COL7">
 <contactref element="R16" pad="1"/>
 <contactref element="U4" pad="6"/>
@@
 <wire x1="31.75" y1="9.525" x2="29.845" y2="7.62" width="0.254" layer="1"/>
 </signal>
-<signal name="N$76">
+<signal name="COL8">
 <contactref element="U4" pad="9"/>
 <contactref element="R17" pad="1"/>
@@
 <wire x1="30.9" y1="11.215" x2="30.9" y2="12.065" width="0.254" layer="1"/>
 </signal>
-<signal name="N$77">
+<signal name="COL9">
 <contactref element="U3" pad="2"/>
 <contactref element="R18" pad="1"/>
@@
 <wire x1="50.38" y1="11.215" x2="50.8" y2="10.795" width="0.254" layer="1"/>
 </signal>
-<signal name="N$78">
+<signal name="COL10">
 <contactref element="U3" pad="4"/>
 <contactref element="R19" pad="1"/>
@@
 <wire x1="48.26" y1="9.525" x2="45.935" y2="9.525" width="0.254" layer="1"/>
 </signal>
-<signal name="N$79">
+<signal name="COL12">
 <contactref element="R21" pad="1"/>
 <contactref element="U3" pad="10"/>
@@
 <wire x1="52.705" y1="9.945" x2="54.19" y2="9.945" width="0.254" layer="1"/>
 </signal>
-<signal name="N$80">
+<signal name="COL11">
 <contactref element="U3" pad="7"/>
 <contactref element="R20" pad="1"/>
@@
 <wire x1="56.73" y1="8.675" x2="55.245" y2="10.16" width="0.254" layer="16"/>
 </signal>
-<signal name="N$81">
+<signal name="COL13">
 <contactref element="R22" pad="1"/>
 <contactref element="U3" pad="1"/>
@@
 <wire x1="67.525" y1="2.54" x2="69.85" y2="2.54" width="0.254" layer="16"/>
 </signal>
-<signal name="N$82">
+<signal name="COL14">
 <contactref element="U3" pad="5"/>
 <contactref element="R23" pad="1"/>
@@
 <wire x1="62.865" y1="6.35" x2="60.96" y2="6.35" width="0.254" layer="16"/>
 </signal>
-<signal name="N$83">
+<signal name="COL15">
 <contactref element="R24" pad="1"/>
 <contactref element="U3" pad="6"/>
@@
 <wire x1="74.08" y1="8.89" x2="68.58" y2="8.89" width="0.254" layer="16"/>
 </signal>
-<signal name="N$84">
+<signal name="COL16">
 <contactref element="U3" pad="9"/>
 <contactref element="R25" pad="1"/>
@@
 <wire x1="57.658" y1="10.16" x2="60.96" y2="10.16" width="0.254" layer="1"/>
 </signal>
-<signal name="N$85">
+<signal name="COL17">
 <contactref element="R26" pad="1"/>
 <contactref element="U2" pad="2"/>
@@
 <wire x1="88.9" y1="7.62" x2="88.9" y2="8.675" width="0.2032" layer="16"/>
 </signal>
-<signal name="N$86">
+<signal name="COL18">
 <contactref element="U2" pad="4"/>
 <contactref element="R27" pad="1"/>
@@
 <wire x1="82.55" y1="8.255" x2="82.55" y2="9.31" width="0.254" layer="16"/>
 </signal>
-<signal name="N$87">
+<signal name="COL19">
 <contactref element="R28" pad="1"/>
 <contactref element="U2" pad="7"/>
@@
 <wire x1="100.115" y1="8.675" x2="100.33" y2="8.89" width="0.254" layer="16"/>
 </signal>
-<signal name="N$88">
+<signal name="COL20">
 <contactref element="U2" pad="10"/>
 <contactref element="R29" pad="1"/>
@@
 <wire x1="93.345" y1="9.945" x2="94.83" y2="9.945" width="0.254" layer="1"/>
 </signal>
-<signal name="N$89">
+<signal name="COL21">
 <contactref element="R30" pad="1"/>
 <contactref element="U2" pad="1"/>
@@
 <wire x1="109.22" y1="4.445" x2="109.22" y2="8.04" width="0.254" layer="16"/>
 </signal>
-<signal name="N$90">
+<signal name="COL22">
 <contactref element="U2" pad="5"/>
 <contactref element="R31" pad="1"/>
@@
 <wire x1="103.632" y1="6.35" x2="103.505" y2="6.35" width="0.254" layer="1"/>
 </signal>
-<signal name="N$91">
+<signal name="COL23">
 <contactref element="R32" pad="1"/>
 <contactref element="U2" pad="6"/>
@@
 <wire x1="106.68" y1="8.89" x2="114.085" y2="8.89" width="0.254" layer="1"/>
 </signal>
-<signal name="N$92">
+<signal name="COL24">
 <contactref element="U2" pad="9"/>
 <contactref element="R33" pad="1"/>
