File: pcb/display-model-a/display.sch (EAGLE design)
At the start: 61 parts, among them J1 SNG-2MM-HEADER-07-V, Q1 ALS-PT19, U1 PIC16F1826-I/SS, U2 74HC4017D, U3 74HC4017D, U4 74HC4017D, U5 74LVC1G08DCKR, U6 74LVC1G08DCKR

Commit message: Changed page format on schematics to US letter (8.5" x 11")
Connections:
- net N$53 renamed COL1
- net N$70 renamed COL2
- net N$71 renamed COL3
- net N$72 renamed COL4
- net N$73 renamed COL5
- net N$74 renamed COL6
- net N$75 renamed COL7
- net N$76 renamed COL8
- net N$77 renamed COL9
- net N$78 renamed COL10
- net N$79 renamed COL12
- net N$80 renamed COL11
- net N$81 renamed COL13
- net N$82 renamed COL14
- net N$83 renamed COL15
- net N$84 renamed COL16
- net N$85 renamed COL17
- net N$86 renamed COL18
- net N$87 renamed COL19
- net N$88 renamed COL20
- net N$89 renamed COL21
- net N$90 renamed COL22
- net N$91 renamed COL23
- net N$92 renamed COL24
