File: pcb/display-model-b/base/base.sch (EAGLE design)
At the start: 48 parts, among them J1 SNG-2MM-HEADER-07-V, Q1 MMBT3904, U1 TSL2561FN, U2 PCA9634PW, U3 74AHC1G04DCK, U4 AP5724W, U5 74AHC1G04DCK, U6 AP5724W, U7 74AHC1G04DCK, U8 AP5724W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

Commit message: Changed page format on schematics to US letter (8.5" x 11")
Other:
- note added: "AMBIENT LIGHT SENSOR"
- note added: "BLUE"
- note added: "GREEN"
- note added: "RED"
