File: pcb/motherboard/audio.sch (KiCad schematic (older format))
At the start: 34 parts, among them J10 HEADER-2x05, J13 DOUT, J14 VOUT-R, J15 GND, U7 PCM2704C, U8 TPA2005, Y1 CRYSTAL

Commit message: Changed crystal location for PCM2704
Parts:
- TP3: value TEST-POINT -> DAC_SHDN
Connections:
- no-connect marks 0 -> 3
Changed lines of the file:
@@
 $EndComp
 $Comp
-L GND #PWR040
+L GND #PWR041
 U 1 1 55016D61
 P 2650 5250
-F 0 "#PWR040" H 2650 5300 30  0001 C CNN
+F 0 "#PWR041" H 2650 5300 30  0001 C CNN
 F 1 "GND" H 2650 5125 30  0001 C CNN
 F 2 "" H 2650 5250 60  0000 C CNN
@@
 $EndComp
 $Comp
-L GND #PWR041
+L GND #PWR042
 U 1 1 55017740
 P 4500 4050
-F 0 "#PWR041" H 4500 4100 30  0001 C CNN
+F 0 "#PWR042" H 4500 4100 30  0001 C CNN
 F 1 "GND" H 4500 3925 30  0001 C CNN
 F 2 "" H 4500 4050 60  0000 C CNN
@@
 $EndComp
 $Comp
-L GND #PWR042
+L GND #PWR043
 U 1 1 55017770
 P 4500 4550
-F 0 "#PWR042" H 4500 4600 30  0001 C CNN
+F 0 "#PWR043" H 4500 4600 30  0001 C CNN
 F 1 "GND" H 4500 4425 30  0001 C CNN
 F 2 "" H 4500 4550 60  0000 C CNN
@@
 $EndComp
 $Comp
-L GND #PWR043
+L GND #PWR044
 U 1 1 55017991
 P 5050 3850
-F 0 "#PWR043" H 5050 3900 30  0001 C CNN
+F 0 "#PWR044" H 5050 3900 30  0001 C CNN
 F 1 "GND" H 5050 3725 30  0001 C CNN
 F 2 "" H 5050 3850 60  0000 C CNN
@@
 $EndComp
 $Comp
-L GND #PWR044
+L GND #PWR045
 U 1 1 550179B3
 P 5450 3700
-F 0 "#PWR044" H 5450 3750 30  0001 C CNN
+F 0 "#PWR045" H 5450 3750 30  0001 C CNN
 F 1 "GND" H 5450 3575 30  0001 C CNN
 F 2 "" H 5450 3700 60  0000 C CNN
@@
 $EndComp
 $Comp
-L GND #PWR045
+L GND #PWR046
 U 1 1 550179CE
 P 5900 3500
-F 0 "#PWR045" H 5900 3550 30  0001 C CNN
+F 0 "#PWR046" H 5900 3550 30  0001 C CNN
 F 1 "GND" H 5900 3375 30  0001 C CNN
 F 2 "" H 5900 3500 60  0000 C CNN
@@
 $EndComp
 $Comp
-L +5V #PWR046
+L +5V #PWR047
 U 1 1 55017A5B
 P 5900 2950
-F 0 "#PWR046" H 5900 3175 30  0001 C CNN
+F 0 "#PWR047" H 5900 3175 30  0001 C CNN
 F 1 "+5V" V 5825 2950 30  0001 C CNN
 F 2 "" H 5900 2950 60  0000 C CNN
@@
 SPK-
 $Comp
-L GND #PWR047
+L GND #PWR048
 U 1 1 5501A691
 P 9550 3350
-F 0 "#PWR047" H 9550 3400 30  0001 C CNN
+F 0 "#PWR048" H 9550 3400 30  0001 C CNN
 F 1 "GND" H 9550 3225 30  0001 C CNN
 F 2 "" H 9550 3350 60  0000 C CNN
@@
 Connection ~ 5900 3050
 Wire Wire Line
-	4300 2850 4850 2850
+	4300 2850 4900 2850
 Connection ~ 3000 4150
 Connection ~ 2650 4750
@@
 Connection ~ 3000 2050
 $Comp
-L GND #PWR048
+L GND #PWR049
 U 1 1 5501B381
 P 2550 1750
-F 0 "#PWR048" H 2550 1800 30  0001 C CNN
+F 0 "#PWR049" H 2550 1800 30  0001 C CNN
 F 1 "GND" H 2550 1625 30  0001 C CNN
 F 2 "" H 2550 1750 60  0000 C CNN
@@
 $EndComp
 $Comp
-L GND #PWR049
+L GND #PWR050
 U 1 1 5501B3B3
 P 5050 1750
-F 0 "#PWR049" H 5050 1800 30  0001 C CNN
+F 0 "#PWR050" H 5050 1800 30  0001 C CNN
 F 1 "GND" H 5050 1625 30  0001 C CNN
 F 2 "" H 5050 1750 60  0000 C CNN
@@
 $EndComp
 $Comp
-L GND #PWR050
+L GND #PWR051
 U 1 1 5501D9CD
 P 5750 5800
-F 0 "#PWR050" H 5750 5850 30  0001 C CNN
+F 0 "#PWR051" H 5750 5850 30  0001 C CNN
 F 1 "GND" H 5750 5675 30  0001 C CNN
 F 2 "" H 5750 5800 60  0000 C CNN
@@
 	6550 4750 6550 5050
 $Comp
-L GND #PWR051
+L GND #PWR052
 U 1 1 5501DF42
 P 6550 5400
-F 0 "#PWR051" H 6550 5450 30  0001 C CNN
+F 0 "#PWR052" H 6550 5450 30  0001 C CNN
 F 1 "GND" H 6550 5275 30  0001 C CNN
 F 2 "" H 6550 5400 60  0000 C CNN
@@
 Connection ~ 7400 5150
 $Comp
-L GND #PWR052
+L GND #PWR053
 U 1 1 5501FEBE
 P 7000 5600
-F 0 "#PWR052" H 7000 5650 30  0001 C CNN
+F 0 "#PWR053" H 7000 5650 30  0001 C CNN
 F 1 "GND" H 7000 5475 30  0001 C CNN
 F 2 "" H 7000 5600 60  0000 C CNN
@@
 $EndComp
 $Comp
-L GND #PWR053
+L GND #PWR054
 U 1 1 55021BA8
 P 8900 5600
-F 0 "#PWR053" H 8900 5650 30  0001 C CNN
+F 0 "#PWR054" H 8900 5650 30  0001 C CNN
 F 1 "GND" H 8900 5475 30  0001 C CNN
 F 2 "" H 8900 5600 60  0000 C CNN
@@
 	8900 5450 8900 5600
 $Comp
-L GND #PWR054
+L GND #PWR055
 U 1 1 55021F7C
 P 10350 5600
-F 0 "#PWR054" H 10350 5650 30  0001 C CNN
+F 0 "#PWR055" H 10350 5650 30  0001 C CNN
 F 1 "GND" H 10350 5475 30  0001 C CNN
 F 2 "" H 10350 5600 60  0000 C CNN
@@
 	10200 4750 10650 4750
 $Comp
-L +5V #PWR055
+L +5V #PWR056
 U 1 1 55023457
 P 8900 3900
-F 0 "#PWR055" H 8900 4125 30  0001 C CNN
+F 0 "#PWR056" H 8900 4125 30  0001 C CNN
 F 1 "+5V" V 8825 3900 30  0001 C CNN
 F 2 "" H 8900 3900 60  0000 C CNN
@@
 $EndComp
 $Comp
-L GND #PWR056
+L GND #PWR057
 U 1 1 55024033
 P 8650 4400
-F 0 "#PWR056" H 8650 4450 30  0001 C CNN
+F 0 "#PWR057" H 8650 4450 30  0001 C CNN
 F 1 "GND" H 8650 4275 30  0001 C CNN
 F 2 "" H 8650 4400 60  0000 C CNN
@@
 $EndComp
 $Comp
-L GND #PWR057
+L GND #PWR058
 U 1 1 55024104
 P 8350 4400
-F 0 "#PWR057" H 8350 4450 30  0001 C CNN
+F 0 "#PWR058" H 8350 4450 30  0001 C CNN
 F 1 "GND" H 8350 4275 30  0001 C CNN
 F 2 "" H 8350 4400 60  0000 C CNN
@@
 DAC_SHDN
 $Comp
-L +5V #PWR058
+L +5V #PWR059
 U 1 1 5502A513
 P 9650 2500
-F 0 "#PWR058" H 9650 2725 30  0001 C CNN
+F 0 "#PWR059" H 9650 2725 30  0001 C CNN
 F 1 "+5V" V 9575 2500 30  0001 C CNN
 F 2 "" H 9650 2500 60  0000 C CNN
@@
 	10150 3050 10650 3050
 Text Label 10550 3050 2    50   ~ 0
-HID1
+HID2
 Wire Wire Line
 	10150 2850 10650 2850
@@
 	9550 2950 9550 3350
 Text Label 10550 2950 2    50   ~ 0
+HID1
+Text Label 10550 2850 2    50   ~ 0
 HID0
-Text Label 10550 2850 2    50   ~ 0
-HID2
 Text Label 9150 2850 0    50   ~ 0
 DAC_SHDN
@@
 P 2350 2750
 F 0 "TP3" H 2300 2825 60  0000 L BNB
-F 1 "TEST-POINT" H 2300 2650 40  0000 L TNN
+F 1 "DAC_SHDN" H 2300 2650 40  0000 L TNN
 F 2 "Conn-Wire-Pads:TEST-POINT-50" H 2200 2725 60  0001 C CNN
 F 3 "" H 2300 2825 60  0001 C CNN
@@
 $EndComp
 $Comp
-L GND #PWR059
+L GND #PWR060
 U 1 1 5509628B
 P 1650 5950
-F 0 "#PWR059" H 1650 6000 30  0001 C CNN
+F 0 "#PWR060" H 1650 6000 30  0001 C CNN
 F 1 "GND" H 1650 5825 30  0001 C CNN
 F 2 "" H 1650 5950 60  0000 C CNN
@@
 Wire Wire Line
 	1650 5750 1650 5950
+NoConn ~ 10150 2750
+NoConn ~ 9750 2750
+NoConn ~ 3100 3350
 $EndSCHEMATC

Commit message: Tidy up motherboard schematic
Parts:
- C14, C15, C16, C17, C18, C19, C21, C25, C26, R10, R11, R12, R13, R14, R4, R5, R6, R7, R8, R9: Family (none) -> Passive
- C20, C27: Family (none) -> Passive; Part (none) -> -; Part# - -> (none)
- C22: value 0.022uF 10V -> 0.022uF (10V); Family (none) -> Passive
- C23, C24: value 100uF 10V -> 100uF (10V); Family (none) -> Passive; Part (none) -> -; Part# - -> (none)
- J10: value HEADER-2x05 -> DF13A-10DP-1.25V; Family (none) -> Connector; MFG (none) -> Hirose
- J13, J14, J15, TP3, TP4: Family (none) -> Virtual
- U7: Family (none) -> IC; MFG (none) -> Analog Devices
- U8: Family (none) -> IC; MFG (none) -> Texas Instruments
- Y1: value CRYSTAL -> 12.00 Mhz; Family (none) -> Passive; PART - -> (none); Part (none) -> -
Changed lines of the file:
@@
 Sheet 3 4
 Title "MOTHERBOARD\\nAUDIO"
-Date "Wed 18 Mar 2015"
+Date "Sun 12 Apr 2015"
 Rev "A"
 Comp ""
@@
 F 2 "SMT-SOP:SSOP28" H 3275 2400 40  0001 C CNN
 F 3 "" H 3200 5300 50  0000 C CNN
+F 4 "IC" H 3700 3850 60  0001 C CNN "Family"
+F 5 "Analog Devices" H 3700 3850 60  0001 C CNN "MFG"
 	1    3700 3850
 	1    0    0    -1
@@
 F 3 "" H 2150 3950 60  0000 C CNN
 F 4 "-" H 2150 4010 45  0001 C CNN "Part"
+F 5 "Passive" H 2150 3850 60  0001 C CNN "Family"
 	1    2150 3850
 	1    0    0    -1
@@
 F 3 "" H 2150 4050 60  0000 C CNN
 F 4 "-" H 2150 4110 45  0001 C CNN "Part"
+F 5 "Passive" H 2150 3950 60  0001 C CNN "Family"
 	1    2150 3950
 	1    0    0    -1
@@
 F 3 "" H 4500 3950 60  0001 C CNN
 F 4 "-" H 4540 4015 45  0001 L CNN "Part"
+F 5 "Passive" H 4500 3850 60  0001 C CNN "Family"
 	1    4500 3850
 	1    0    0    -1
@@
 F 3 "" H 4500 4450 60  0001 C CNN
 F 4 "-" H 4540 4515 45  0001 L CNN "Part"
+F 5 "Passive" H 4500 4350 60  0001 C CNN "Family"
 	1    4500 4350
 	1    0    0    -1
@@
 F 3 "" H 5050 3800 60  0001 C CNN
 F 4 "-" H 5090 3865 45  0001 L CNN "Part"
+F 5 "Passive" H 5050 3700 60  0001 C CNN "Family"
 	1    5050 3700
 	1    0    0    -1
@@
 F 2 "SMT:CPL-0805" H 5485 3345 40  0001 L CNN
 F 3 "" H 5450 3600 60  0000 C CNN
-F 4 "-" H 5485 3665 45  0001 L CNN "Part#"
+F 4 "-" H 5485 3665 45  0001 L CNN "Part"
+F 5 "Passive" H 5450 3500 60  0001 C CNN "Family"
 	1    5450 3500
 	1    0    0    -1
@@
 F 3 "" H 5900 3400 60  0001 C CNN
 F 4 "-" H 5940 3465 45  0001 L CNN "Part"
+F 5 "Passive" H 5900 3300 60  0001 C CNN "Family"
 	1    5900 3300
 	1    0    0    -1
@@
 F 3 "" H 2650 4550 60  0001 C CNN
 F 4 "-" H 2690 4615 45  0001 L CNN "Part"
+F 5 "Passive" H 2650 4450 60  0001 C CNN "Family"
 	1    2650 4450
 	1    0    0    -1
@@
 F 3 "" H 1800 3750 60  0000 C CNN
 F 4 "-" H 1800 3810 45  0001 C CNN "Part"
+F 5 "Passive" H 1800 3650 60  0001 C CNN "Family"
 	1    1800 3650
 	0    -1   1    0
@@
 F 3 "" H 2150 3550 60  0000 C CNN
 F 4 "-" H 2150 3610 45  0001 C CNN "Part"
+F 5 "Passive" H 2150 3450 60  0001 C CNN "Family"
 	1    2150 3450
 	1    0    0    -1
@@
 F 3 "" H 3700 2150 60  0000 C CNN
 F 4 "-" H 3700 2210 45  0001 C CNN "Part"
+F 5 "Passive" H 3700 2050 60  0001 C CNN "Family"
 	1    3700 2050
 	1    0    0    -1
@@
 P 9950 2950
 F 0 "J10" H 9850 3250 60  0000 L BNB
-F 1 "HEADER-2x05" H 9850 2650 40  0001 L TNN
+F 1 "DF13A-10DP-1.25V" H 9850 2650 40  0000 L TNN
 F 2 "Conn-Hirose:DF13A-10DP-1.25" H 9950 1750 60  0001 C CNN
 F 3 "" H 9950 1750 60  0001 C CNN
+F 4 "Connector" H 9950 2950 60  0001 C CNN "Family"
+F 5 "Hirose" H 9950 2650 40  0001 C CNN "MFG"
 	1    9950 2950
 	1    0    0    -1
@@
 P 3700 1650
 F 0 "Y1" H 3700 1760 60  0000 C CNB
-F 1 "CRYSTAL" H 3700 1550 40  0000 C CNN
+F 1 "12.00 Mhz" H 3700 1550 40  0000 C CNN
 F 2 "Crystals:HC49UP" H 3700 1490 40  0001 C CNN
 F 3 "" H 3700 1770 60  0000 C CNN
-F 4 "-" H 3705 1825 45  0001 C CNN "PART"
+F 4 "-" H 3705 1825 45  0001 C CNN "Part"
+F 5 "Passive" H 3700 1650 60  0001 C CNN "Family"
 	1    3700 1650
 	1    0    0    -1
@@
 F 3 "" H 2750 1750 60  0001 C CNN
 F 4 "-" H 2790 1815 45  0001 L CNN "Part"
+F 5 "Passive" H 2750 1650 60  0001 C CNN "Family"
 	1    2750 1650
 	0    -1   -1   0
@@
 F 3 "" H 4800 1750 60  0001 C CNN
 F 4 "-" H 4840 1815 45  0001 L CNN "Part"
+F 5 "Passive" H 4800 1650 60  0001 C CNN "Family"
 	1    4800 1650
 	0    -1   -1   0
@@
 P 5750 5150
 F 0 "C22" H 5780 5240 60  0000 L CNB
-F 1 "0.022uF 10V" H 5780 5060 45  0000 L CNN
+F 1 "0.022uF (10V)" H 5780 5060 45  0000 L CNN
 F 2 "SMT:C-0603" H 5785 4995 40  0001 L CNN
 F 3 "" H 5750 5250 60  0001 C CNN
 F 4 "-" H 5790 5315 45  0001 L CNN "Part"
+F 5 "Passive" H 5750 5150 60  0001 C CNN "Family"
 	1    5750 5150
 	1    0    0    -1
@@
 F 3 "" H 5750 5650 60  0000 C CNN
 F 4 "-" H 5750 5710 45  0001 C CNN "Part"
+F 5 "Passive" H 5750 5550 60  0001 C CNN "Family"
 	1    5750 5550
 	0    -1   -1   0
@@
 P 6150 4750
 F 0 "C23" H 6180 4840 60  0000 L CNB
-F 1 "100uF 10V" H 6180 4660 45  0000 L CNN
+F 1 "100uF (10V)" H 6180 4660 45  0000 L CNN
 F 2 "SMT:CPL-1210" H 6185 4595 40  0001 L CNN
 F 3 "" H 6150 4850 60  0000 C CNN
-F 4 "-" H 6185 4915 45  0001 L CNN "Part#"
+F 4 "-" H 6185 4915 45  0001 L CNN "Part"
+F 5 "Passive" H 6150 4750 60  0001 C CNN "Family"
 	1    6150 4750
 	0    -1   -1   0
@@
 F 3 "" H 6550 5250 60  0000 C CNN
 F 4 "-" H 6550 5310 45  0001 C CNN "Part"
+F 5 "Passive" H 6550 5150 60  0001 C CNN "Family"
 	1    6550 5150
 	0    -1   -1   0
@@
 P 6850 4750
 F 0 "C24" H 6900 4650 60  0000 L CNB
-F 1 "100uF 10V" H 6900 4850 45  0000 L CNN
+F 1 "100uF (10V)" H 6900 4850 45  0000 L CNN
 F 2 "SMT:CPL-0805" H 6885 4595 40  0001 L CNN
 F 3 "" H 6850 4850 60  0000 C CNN
-F 4 "-" H 6885 4915 45  0001 L CNN "Part#"
+F 4 "-" H 6885 4915 45  0001 L CNN "Part"
+F 5 "Passive" H 6850 4750 60  0001 C CNN "Family"
 	1    6850 4750
 	0    1    -1   0
@@
 F 3 "" H 7700 4850 60  0000 C CNN
 F 4 "-" H 7700 4910 45  0001 C CNN "Part"
+F 5 "Passive" H 7700 4750 60  0001 C CNN "Family"
 	1    7700 4750
 	1    0    0    -1
@@
 F 3 "" H 7700 4500 60  0000 C CNN
 F 4 "-" H 7700 4560 45  0001 C CNN "Part"
+F 5 "Passive" H 7700 4400 60  0001 C CNN "Family"
 	1    7700 4400
 	1    0    0    -1
@@
 F 3 "" H 7700 5250 60  0000 C CNN
 F 4 "-" H 7700 5310 45  0001 C CNN "Part"
+F 5 "Passive" H 7700 5150 60  0001 C CNN "Family"
 	1    7700 5150
 	1    0    0    -1
@@
 F 3 "" H 7700 5650 60  0000 C CNN
 F 4 "-" H 7700 5710 45  0001 C CNN "Part"
+F 5 "Passive" H 7700 5550 60  0001 C CNN "Family"
 	1    7700 5550
 	1    0    0    -1
@@
 F 3 "" H 7000 5500 60  0001 C CNN
 F 4 "-" H 7040 5565 45  0001 L CNN "Part"
+F 5 "Passive" H 7000 5400 60  0001 C CNN "Family"
 	1    7000 5400
 	1    0    0    -1
@@
 F 2 "SMT-SOP:PPSOP8" H 9175 4300 40  0001 C CNN
 F 3 "" H 9100 5600 50  0000 C CNN
+F 4 "IC" H 9600 5000 60  0001 C CNN "Family"
+F 5 "Texas Instruments" H 9600 5000 60  0001 C CNN "MFG"
 	1    9600 5000
 	1    0    0    -1
@@
 F 2 "SMT:CPL-0805" H 8685 4095 40  0001 L CNN
 F 3 "" H 8650 4350 60  0000 C CNN
-F 4 "-" H 8685 4415 45  0001 L CNN "Part#"
+F 4 "-" H 8685 4415 45  0001 L CNN "Part"
+F 5 "Passive" H 8650 4250 60  0001 C CNN "Family"
 	1    8650 4250
 	1    0    0    -1
@@
 F 3 "" H 8350 4350 60  0001 C CNN
 F 4 "-" H 8390 4415 45  0001 L CNN "Part"
+F 5 "Passive" H 8350 4250 60  0001 C CNN "Family"
 	1    8350 4250
 	1    0    0    -1
@@
 F 2 "Conn-Wire-Pads:WP-50mil-1x01" H 2500 3625 60  0001 C CNN
 F 3 "" H 2600 3725 60  0001 C CNN
+F 4 "Virtual" H 2650 3650 60  0001 C CNN "Family"
 	1    2650 3650
 	-1   0    0    1
@@
 F 2 "Conn-Wire-Pads:WP-50mil-1x01" H 4750 5025 60  0001 C CNN
 F 3 "" H 4850 5125 60  0001 C CNN
+F 4 "Virtual" H 4900 5050 60  0001 C CNN "Family"
 	1    4900 5050
 	1    0    0    -1
@@
 F 2 "Conn-Wire-Pads:TEST-POINT-50" H 5600 4375 60  0001 C CNN
 F 3 "" H 5700 4475 60  0001 C CNN
+F 4 "Virtual" H 5750 4400 60  0001 C CNN "Family"
 	1    5750 4400
 	0    -1   -1   0
@@
 F 2 "Conn-Wire-Pads:TEST-POINT-50" H 2200 2725 60  0001 C CNN
 F 3 "" H 2300 2825 60  0001 C CNN
+F 4 "Virtual" H 2350 2750 60  0001 C CNN "Family"
 	1    2350 2750
 	-1   0    0    -1
@@
 F 2 "Conn-Wire-Pads:WP-50mil-1x01" H 1500 5575 60  0001 C CNN
 F 3 "" H 1600 5675 60  0001 C CNN
+F 4 "Virtual" H 1650 5600 60  0001 C CNN "Family"
 	1    1650 5600
 	0    -1   -1   0
