File: pcb/left-panel/left-panel.sch (KiCad schematic (older format))
At the start: 6 parts, among them J1 DF3A-4P-2DSA, SW1 B3F-3150, SW2 B3F-3150, SW3 B3F-3150

Commit message: Added components count on CLK-PC-03 BOM
Parts:
- H1, H2: Family (none) -> Virtual
- J1: Family (none) -> Connector; MFG (none) -> Hirose
- SW1, SW2, SW3: Family (none) -> Switch
Changed lines of the file:
@@
 F 2 "Conn-Hirose:DF3A-4P-2DSA" H 6500 5050 60  0001 C CNN
 F 3 "" H 6500 5050 60  0001 C CNN
+F 4 "Connector" H 6500 5050 60  0001 C CNN "Family"
+F 5 "Hirose" H 6500 5050 60  0001 C CNN "MFG"
 	1    6500 5050
 	1    0    0    -1
@@
 F 2 "Switches:B3F-315X" H 5125 2325 40  0001 L TNN
 F 3 "" H 4950 2600 60  0001 C CNN
+F 4 "Switch" H 5050 2500 60  0001 C CNN "Family"
 	1    5050 2500
 	1    0    0    -1
@@
 F 2 "Switches:B3F-315X" H 5125 3075 40  0001 L TNN
 F 3 "" H 4950 3350 60  0001 C CNN
+F 4 "Switch" H 5050 3250 60  0001 C CNN "Family"
 	1    5050 3250
 	1    0    0    -1
@@
 F 2 "Switches:B3F-315X" H 5125 3775 40  0001 L TNN
 F 3 "" H 4950 4050 60  0001 C CNN
+F 4 "Switch" H 5050 3950 60  0001 C CNN "Family"
 	1    5050 3950
 	1    0    0    -1
@@
 F 2 "Conn-Wire-Pads:Hole-Screw-NP-#4" H 8500 1625 40  0001 L TNN
 F 3 "" H 8400 1875 60  0001 C CNN
+F 4 "Virtual" H 8450 1800 60  0001 C CNN "Family"
 	1    8450 1800
 	1    0    0    -1
@@
 F 2 "Conn-Wire-Pads:Hole-Screw-NP-#4" H 8950 1625 40  0001 L TNN
 F 3 "" H 8850 1875 60  0001 C CNN
+F 4 "Virtual" H 8900 1800 60  0001 C CNN "Family"
 	1    8900 1800
 	1    0    0    -1
